File: Kicad/SCAN-2000-LV-20.sch (KiCad schematic (older format))
At the start: 191 parts, among them J1 FTDI, J10 OUTPUT-BUS-A, J11 OUTPUT-BUS-B, J12 Test, J13 Conn_02x04_Counter_Clockwise, J2 Conn_01x02, J3 Conn_01x02, J4 BUS-A-INPUT, J5 SWD, J6 BUS-A-INPUT, J7 BUS-B-INPUT, J8 BUS-B-INPUT, J9 MOLEX 85050-0000, K1 EC2-3TNU, U1 STM32G030, U10 DG412, U11 DG412, U12 RB-0515D, U13 MDC3105, U14 TPS78233DDC, U15 TL7733BD, U16 MDC3105, U17 RB-0505S, U2 DG412, U3 DG412, U4 DG412, U5 DG412, U6 DG412, U7 DG412, U8 DG412, U9 DG412

Commit message: Board layout for the Switches
Parts:
- removed C13, C15, C17, C18, C19, C20, C21, C25, C27, C30, C32, C34, C35, C36, C37, C38, C40, C42: 0.1u, Capacitors-SMD:C_0805_2012Metric_Pad1.18x1.45mm_HandSolder, symbol Device:C
- removed C44: 10u, Capacitors-SMD:C_0805_2012Metric_Pad1.18x1.45mm_HandSolder, symbol Device:C
- removed C45: 1u, Capacitors-SMD:C_0805_2012Metric_Pad1.18x1.45mm_HandSolder, symbol Device:C
- removed D1, D10, D11, D12, D13, D14, D2, D3, D4, D5, D6, D7, D8, D9: BAV199L, SMD-SOT:SOT-23, symbol Diode:BAV99
- removed L3: L, Inductor_SMD:L_0805_2012Metric_Pad1.15x1.40mm_HandSolder, symbol Device:L
- removed R? (x40): 200R, Resistors-SMD:R_2512_6332Metric_Pad1.40x3.35mm_HandSolder, symbol Device:R
- removed U10, U11, U2, U3, U4, U5, U6, U7, U8, U9: DG412, SMD-SO:SOIC-16_3.9x9.9mm_P1.27mm, symbol Analog_Switch:DG412xY
- removed U17: RB-0505S, DC-DC-Module:RB-0515D, symbol DC-DC~Power~Modules:CMR0515S3C
- added D1, D2: LED, Resistors-SMD:R_0805_2012Metric_Pad1.20x1.40mm_HandSolder, symbol Device:LED
- added D10, D11, D12, D13, D14, D3, D4, D5, D6, D7, D8, D9: D, Resistors-SMD:R_0805_2012Metric_Pad1.20x1.40mm_HandSolder, symbol Device:D
- added D45, D46, D47, D48, D49, D50, D51, D52, D53, D54, D55, D56, D57, D58: BAV199, Package_TO_SOT_SMD:SOT-23, symbol Diode:BAV99
- added R100, R101, R102, R103, R104, R105, R106, R67, R68, R69, R70, R71, R72, R73, R74, R75, R76, R77, R78, R79, R80, R81, R82, R83, R84, R85, R86, R87, R88, R89, R90, R91, R92, R93, R94, R95, R96, R97, R98, R99: 200R, Resistors-SMD:R_0805_2012Metric_Pad1.20x1.40mm_HandSolder, symbol Device:R
- added R25, R26: R, Resistors-SMD:R_0805_2012Metric_Pad1.20x1.40mm_HandSolder, symbol Device:R
- added U2, U3, U4, U5, U6, U7: DG409, SMD-SO:SOIC-16_3.9x9.9mm_P1.27mm, symbol DG509ACWE:DG509ACWE
- D15, D16, D17, D18, D19, D20, D21, D22, D23, D24, D25, D26, D27, D28, D29, D30, D31, D32, D33, D34, D35, D36, D37, D38, D39, D40: value BAV199L -> BAV199; footprint SMD-SOT:SOT-23 -> Package_TO_SOT_SMD:SOT-23
- U12: symbol DC-DC~Power~Modules:CMR0515S3C -> SCAN-2000-LV-20-rescue:CMR0515S3C-DC-DC_Power_Modules
- U13, U16: symbol Relay~Drivers~K:MDC3105 -> SCAN-2000-LV-20-rescue:MDC3105-Relay_Drivers_K
Connections:
- net labels added: CON-A0-DIG, CON-A1-DIG, EN-U2-DIG, EN-U3-DIG, EN-U4-DIG, EN-U5-DIG, EN-U6-DIG, EN-U7-Dig
- net labels removed: +VDC, CHAN-01A-CON, CHAN-01B-CON, CHAN-02A-CON, CHAN-02B-CON, CHAN-03A-CON, CHAN-03B-CON, CHAN-04A-CON, CHAN-04B-CON, CHAN-05A-CON, CHAN-05B-CON, CHAN-06A-CON, CHAN-06B-CON, CHAN-07A-CON, CHAN-07B-CON, CHAN-08A-CON, CHAN-08B-CON, CHAN-09A-CON, CHAN-09B-CON, CHAN-10A-CON, CHAN-10B-CON
- wire segments 1018 -> 708
- no-connect marks 2 -> 17
Other:
- note added: "DG409 Bypass"
- note removed: "Isolated Input"
- moved on the sheet: C1, C10, C11, C12, C14, C16, C2, C22, C23, C24, C26, C28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
